Commit message: VLP-16을 베이스로 RDV-128생성( 128ch, FOV 105' )

File: velodyne_description/urdf/example.urdf.xacro (robot description, xacro)
@@ -30,4 +30,9 @@
     </inertial>
   </link>
+  <xacro:include filename="$(find velodyne_description)/urdf/RDV-128.urdf.xacro"/>
+  <xacro:RDV-128 parent="base_link" name="velodyne" topic="/velodyne_points" hz="10" samples="440" gpu="${gpu}">
+    <origin xyz="0 0 0.4" rpy="0 0 0" />
+  </xacro:RDV-128>
+  <!--
   <xacro:include filename="$(find velodyne_description)/urdf/VLP-16.urdf.xacro"/>
   <xacro:VLP-16 parent="base_link" name="velodyne" topic="/velodyne_points" hz="10" samples="440" gpu="${gpu}">
@@ -38,3 +43,4 @@
     <origin xyz="0 0 0.6" rpy="0 0 0" />
   </xacro:HDL-32E>
+  -->
 </robot>
